File: hardware/swadge2019.kicad_pcb (KiCad board)
At the start: 2 copper layers, 100 x 95.3 mm, 50 parts, among them P1 PGM, P10 CONN_1, P11 CONN_1, P12 CONN_1, P13 CONN_1, P2 USBMicroB-10118192-0001LF, P3 SAO, P7 CONN_1, P8 CONN_1, P9 CONN_1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

Commit message: Rescued schematic, started adding 3D models to layout
Parts:
- BT1, BT2: footprint BCAAPC -> Swadge_Parts:2460
- C1, C2, C3, C4, C5, C6, C7, C8: footprint C_0805 -> Swadge_Parts:C_0805_2012Metric
- ESP1: footprint ESP12E -> Swadge_Parts:ESP12E
- R1, R10, R11, R2, R3, R4, R5, R6, R7, R8, R9: footprint R_0805 -> Swadge_Parts:R_0805_2012Metric
- SW1, SW2: footprint TACTILE10 -> Swadge_Parts:SW_4-1437565-2
- SW3: footprint TACT_3x6_SINGLE -> Swadge_Parts:TACT_3x6_SINGLE
- U1: footprint SOT-23-5 -> Swadge_Parts:SOT-23-5
- U2: footprint SOT-223 -> Swadge_Parts:SOT-223-3_TabPin2
- Y1: footprint C_Radial_D8_L13_P3.8 -> Swadge_Parts:C_Radial_D8_L13_P3.8
- turned BT1 to 0 degrees
- turned BT2 to 180 degrees
- turned U2 to 90 degrees
