File: hardware/swadge2019.kicad_pcb (KiCad board)
At the start: 2 copper layers, 100 x 95.3 mm, 51 parts, among them P1 PGM, P10 CONN_1, P11 CONN_1, P12 CONN_1, P13 CONN_1, P2 USB_Micro-B_Molex_47346-0001, P3 SAO, P7 CONN_1, P8 CONN_1, P9 CONN_1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

Commit message: Added cube for LEDs
Parts:
- D1, D2, D3, D4, D5, D6: footprint charles:SK6812SIDE -> Swadge_Parts:SK6812SIDE
- moved P2 0.69 mm to (61.5, 124.8)
Routing:
- net GND: track 320.9 -> 310.0 mm
